Commit message: Updated forward kinematics for z

File: scara_pkg_gr03/model/ms2r1p_amg.urdf.xacro (robot description, xacro)
@@ -3,5 +3,5 @@
     <!--Propiedades-->
     <xacro:property name="rescale" value="${1000}" />
-    <xacro:property name="r1" value="1.60" />
+    <xacro:property name="r1" value="${1.60/10}" />
     <xacro:property name="base_x" value="${200/rescale}" />
     <xacro:property name="base_y" value="${139/rescale}" />

Commit message: Fixed xacro: prismatic joint matches real life

File: scara_pkg_gr03/model/ms2r1p_amg.urdf.xacro (robot description, xacro)
@@ -110,5 +110,5 @@
         <parent link="arm_2_link"/>
         <child link="prismatic_link"/>
-        <origin xyz="${arm_2_x-off_edge_center_arm2-prism_r-off_edge_prism_arm2} 0 ${-0.006}" rpy="0 0 0"/>
+        <origin xyz="${arm_2_x-off_edge_center_arm2-prism_r-off_edge_prism_arm2} 0 ${-0.011}" rpy="0 0 0"/>
         <axis xyz="0 0 -1"/>
         <limit effort="1" lower="${lower_limit_linear}" upper="${upper_limit_linear}" velocity="1"/>
@@ -123,4 +123,5 @@
                 <color rgba="0.5 0.5 0.5 0.8"/> <!-- R G B A -->
             </material>
+            <!-- Visual origin adjusted: cylinder bottom should align with joint origin -->
             <origin xyz="0 0 ${prism_len/2}" rpy="0 0 0"/>
         </visual>
@@ -134,5 +135,5 @@
                    <cylinder radius="${prism_r}" length="${prism_len}"/>
                 </geometry>
-                <origin xyz="0 0 ${prism_len/2}" rpy="0 0 0"/>
+                <origin xyz="0 0 ${-prism_len/2}" rpy="0 0 0"/>
             </collision>
     </link>
